File: cy8c5287axi_board/cy8c5287axi_board.kicad_pcb (KiCad board)
At the start: 2 copper layers, 68 parts, among them CON1 USB-MINI-B, P1 CONN_2, P2 CONN_2, P3 CONN_1, P4 CONN_1, P5 CONN_1, P6 CONN_1, SW1 SW_PUSH, SW2 SW_PUSH, U1 CY8C52LP_100TQFP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

Commit message: Create
Parts:
- removed IO_CapSense1, IO_USB1: CONN_2, PIN_ARRAY_2X1
- removed Prog_JTAG1: CONN_5X2, PIN_ARRAY_5x2
- removed Prog_SWD1: CONN_5, PIN_ARRAY_5x1
- removed R10, R9: 0, SM0603
- added IO_CapSense: , PIN_ARRAY_2X1, F.Cu at (80.2, 48.2)
- added Prog_JTAG: , PIN_ARRAY_5x2, F.Cu at (63.0, 36.0)
- added Prog_SWD: , PIN_ARRAY_5x1, F.Cu at (80.8, 34.8)
- added R21: 0, SM0603, F.Cu at (105.5, 76.5)
- added R22: 0, SM0603, F.Cu at (105.5, 72.0)
- added VDDA: , SM0603_Contact, B.Cu at (86.9, 89.7)
- added VSSA: , SM0603_Contact, B.Cu at (86.9, 87.6)
- ?: renamed from P1; value CONN_2 -> VDD<-VPROG
- ?: renamed from P6; value CONN_1 -> (none)
- ?: renamed from P5; value CONN_1 -> (none)
- ?: renamed from P4; value CONN_1 -> (none)
- ?: renamed from P3; value CONN_1 -> (none)
- C1, C10, C11, C12, C16, C17, C2, C6, C8, C9, R15, R16, R17, R18, R19, R20: moved to B.Cu
- D3: value DIODESCH -> SBD
- D4: value LED -> LED(2.1)
- D5: value LED -> LED(2.2)
- IO1, IO2: value CONN_30 -> (none)
- IO_LED: renamed from IO_LED1; value CONN_4 -> (none)
- IO_Power: renamed from IO_Power1; value CONN_4X2 -> (none)
- IO_SAR: renamed from IO_SAR1; value CONN_4 -> (none)
- R4: value R -> (none)
- SW(2.4): renamed from SW2; value SW_PUSH -> (none)
- SW1(2.3): renamed from SW1; value SW_PUSH -> (none)
- VUSB->VDD: renamed from P2; value CONN_2 -> (none)
- moved R11 121.9 mm to (90.2, 82.0), turned to 270 degrees
- moved R12 116.7 mm to (97.3, 64.5)
- moved R13 115.6 mm to (97.3, 62.5)
- moved R14 111.8 mm to (93.2, 61.7)
- moved R17 110.4 mm to (98.5, 49.8)
- moved R18 109.1 mm to (98.5, 47.0)
- moved R19 108.1 mm to (98.5, 44.5)
- moved R20 107.1 mm to (98.5, 42.0)
- moved R15 97.8 mm to (80.0, 56.2), turned to 180 degrees
- moved R16 95.8 mm to (80.2, 52.2), turned to 90 degrees
- moved C13 76.2 mm to (72.8, 47.2), turned to 0 degrees
- moved IO_Power 67.8 mm to (72.2, 98.0), turned to 0 degrees
- moved R4 59.8 mm to (69.8, 92.0), turned to 0 degrees
- moved IO_LED 54.4 mm to (110.8, 45.8), turned to 90 degrees
- moved ? 54.3 mm to (74.8, 92.0)
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- renumbered CON1 to ?, X1 to ?, D2 to ?
Connections:
- ? pad 1: /15.2* -> /kHz_XO
- ? pad 2: /15.3* -> /kHz_XI
- C19 pad 1: /15.2* -> /kHz_XO
- C20 pad 1: /15.3* -> /kHz_XI
- U1 pad 55: /15.2* -> /kHz_XO
- U1 pad 56: /15.3* -> /kHz_XI
Routing:
- net VSSD: track 49.2 -> 665.6 mm, vias 6 -> 101
- net VDDD: track 91.0 -> 198.0 mm, vias 2 -> 32
- net /1.1: track 0.00 -> 100.5 mm, vias 0 -> 2
- net /1.0: track 0.00 -> 93.2 mm, vias 0 -> 2
- net //XRES: track 0.00 -> 89.3 mm, vias 0 -> 1
- net /1.4: track 0.00 -> 79.2 mm, vias 0 -> 1
- net VPROG: track 0.00 -> 78.6 mm, vias 0 -> 6
- net /1.3: track 0.00 -> 75.7 mm, vias 0 -> 1
- net /3.0: track 0.00 -> 67.0 mm, vias 0 -> 2
- net /2.0: track 0.00 -> 64.5 mm
- net /15.1: track 0.00 -> 62.8 mm, vias 0 -> 2
- net /3.1: track 0.00 -> 61.3 mm
- net /6.3: track 0.00 -> 59.4 mm
- net /15.0: track 0.00 -> 58.8 mm, vias 0 -> 2
- net VSSA: track 12.4 -> 69.6 mm
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- added copper zone on F.Cu, net VSSD
- removed copper zone on F.Cu, net N-0000095
- removed copper zone on B.Cu, net VSSA
Other:
- board outline added: 80 x 100 mm
- board text added: "15.4 15.5"
- board text added: "2.0 6.3 6.2 6.1 6.0 4.7 4.6 4.5 4.4 4.3 4.2 0.7 0.6 0.5 0.1 0.0 4.1 4.0 12.3 12.2 *15.3 *15.2 12.1 12.0 3.7 3.6 3.5 3.4 3.3 3.1"
- board text added: "2.4 2.3 2.2 2.1"
- board text added: "2.5 2.6 2.7 12.4 12.5 6.4 6.5 6.6 6.7 5.0 5.1 5.2 5.3 1.0 1.1 1.2 1.3 1.4 1.5 1.6 1.7 12.6 12.7 5.4 5.5 5.6 5.7 15.0 15.1 3.0"
- board text added: "2015 08/01 Rev.A"
- board text added: "3.2 0.2 0.3 0.4"
- board text added: "CYPRESS CY8C52LP Evaluation Board"
- board text added: "CapSense or GPIO"
- board text added: "Designed by Fumiya Katoh"
- board text added: "GND"
- board text added: "GND GND GND GND VPROG"
- board text added: "GND VDD"
- board text added: "OnBoard SW/LED or GPIO"
- board text added: "RESET TDI TDO TCK TMS"
- board text added: "SAR_ADC or GPIO"
- board text added: "VDD"
- board text added: "VPROG GND XRES SWDCK SWDIO"
- board text added: "XTAL or GPIO"
