File: cy8c5287axi_board/cy8c5287axi_board.sch (KiCad schematic (older format))
At the start: 68 parts, among them CON1 USB-MINI-B, P1 CONN_2, P2 CONN_2, P3 CONN_1, P4 CONN_1, P5 CONN_1, P6 CONN_1, SW1 SW_PUSH, SW2 SW_PUSH, U1 CY8C52LP_100TQFP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

Commit message: Create
Parts:
- removed IO_USB1: CONN_2, ~, symbol CONN_2
- added R21, R22: 0, ~, symbol R
Other:
- note removed: "USB\n"
- moved on the sheet: IO_CapSense1, IO_LED1, IO_SAR1, R11, R12, R13, R14, R15, R16, R17, R18, R19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
