File: rev_b.kicad_pcb (KiCad board)
At the start: 2 copper layers, 50 x 50 mm, 86 parts, among them CON1 USB-MINI-B, P1 CONN_3X2, P10 CONN_10X2, P11 CONN_BATT, P12 CONN_4, P13 CONN_4, P3 CONN_1, P4 CONN_1, P5 CONN_1, P6 CONN_1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

Commit message: Fixed: ReturnPass
Routing:
- net VSSD: track 494.7 -> 561.6 mm, vias 66 -> 73
- net N-0000088: track 29.5 -> 27.9 mm, vias 2 -> 1
- net /5.6: track 17.5 -> 18.1 mm
- net /15.0*: track 43.4 -> 43.9 mm
- net //XRES: track 26.0 -> 26.4 mm, vias 1 -> 2
Other:
- board text added: "5V PROG 3.3V"
- board text added: "Rev.B"
- board text removed: "5V VPROG 3.3V"
- board text removed: "by F.Katoh"
